File: pcb/shutter_tester.sch (KiCad schematic (older format))
At the start: 16 parts, among them J1 Conn_01x04, Q1 MMBTA13LT3G, U1 LM393

Commit message: add pulldown resistor to darlington
Parts:
- added R7: 4.7M, Resistor_SMD:R_0603_1608Metric_Pad0.98x0.95mm_HandSolder, symbol Device:R
- D1: footprint LED_SMD:LED_0603_1608Metric_Pad1.05x0.95mm_HandSolder -> LED_SMD:LED_0805_2012Metric_Pad1.15x1.40mm_HandSolder
- R5: value 4.7M -> 102k
- gave numbers to parts that had none: 1
Connections:
- net GND: now also R7.2
- net at D1.2 (A), Q1.1 (B): now also R7.1
Other:
- moved on the sheet: C1, U1B, U1C
Changed lines of the file:
@@
 F 0 "D1" H 3300 3250 50  0000 C CNN
 F 1 "LED" H 3300 3050 50  0000 C CNN
-F 2 "LED_SMD:LED_0603_1608Metric_Pad1.05x0.95mm_HandSolder" H 3300 3150 50  0001 C CNN
+F 2 "LED_SMD:LED_0805_2012Metric_Pad1.15x1.40mm_HandSolder" H 3300 3150 50  0001 C CNN
 F 3 "~" H 3300 3150 50  0001 C CNN
 	1    3300 3150
@@
 L power:GND #PWR04
 U 1 1 61238FED
-P 3700 3900
-F 0 "#PWR04" H 3700 3650 50  0001 C CNN
-F 1 "GND" H 3700 3750 50  0000 C CNN
-F 2 "" H 3700 3900 50  0001 C CNN
-F 3 "" H 3700 3900 50  0001 C CNN
-	1    3700 3900
-	1    0    0    -1
-$EndComp
-Wire Wire Line
-	3700 3900 3700 3800
+P 3700 4050
+F 0 "#PWR04" H 3700 3800 50  0001 C CNN
+F 1 "GND" H 3700 3900 50  0000 C CNN
+F 2 "" H 3700 4050 50  0001 C CNN
+F 3 "" H 3700 4050 50  0001 C CNN
+	1    3700 4050
+	1    0    0    -1
+$EndComp
+Wire Wire Line
+	3700 4050 3700 3800
 $Comp
 L power:GND #PWR07
 U 1 1 61238FFA
-P 5150 3850
-F 0 "#PWR07" H 5150 3600 50  0001 C CNN
-F 1 "GND" H 5150 3700 50  0000 C CNN
-F 2 "" H 5150 3850 50  0001 C CNN
-F 3 "" H 5150 3850 50  0001 C CNN
-	1    5150 3850
-	1    0    0    -1
-$EndComp
-Wire Wire Line
-	5150 3850 5150 3800
+P 5150 4050
+F 0 "#PWR07" H 5150 3800 50  0001 C CNN
+F 1 "GND" H 5150 3900 50  0000 C CNN
+F 2 "" H 5150 4050 50  0001 C CNN
+F 3 "" H 5150 4050 50  0001 C CNN
+	1    5150 4050
+	1    0    0    -1
+$EndComp
+Wire Wire Line
+	5150 4050 5150 3800
 $Comp
 L Device:Q_NPN_Darlington_BEC Q1
@@
 L Comparator:LM393 U1
 U 2 1 61691692
-P 4650 4800
-F 0 "U1" H 4800 4950 50  0000 C CNN
-F 1 "LM393" H 4900 4650 50  0000 C CNN
-F 2 "Package_SO:SOP-8_3.9x4.9mm_P1.27mm" H 4650 4800 50  0001 C CNN
-F 3 "http://www.ti.com/lit/ds/symlink/lm393.pdf" H 4650 4800 50  0001 C CNN
-	2    4650 4800
+P 4650 5000
+F 0 "U1" H 4800 5150 50  0000 C CNN
+F 1 "LM393" H 4900 4850 50  0000 C CNN
+F 2 "Package_SO:SOP-8_3.9x4.9mm_P1.27mm" H 4650 5000 50  0001 C CNN
+F 3 "http://www.ti.com/lit/ds/symlink/lm393.pdf" H 4650 5000 50  0001 C CNN
+	2    4650 5000
 	1    0    0    -1
 $EndComp
@@
 L Comparator:LM393 U1
 U 3 1 61691D9C
-P 3800 4650
-F 0 "U1" H 3950 4800 50  0000 C CNN
-F 1 "LM393" H 4050 4500 50  0000 C CNN
-F 2 "Package_SO:SOP-8_3.9x4.9mm_P1.27mm" H 3800 4650 50  0001 C CNN
-F 3 "http://www.ti.com/lit/ds/symlink/lm393.pdf" H 3800 4650 50  0001 C CNN
-	3    3800 4650
+P 3800 4850
+F 0 "U1" H 3950 5000 50  0000 C CNN
+F 1 "LM393" H 4050 4700 50  0000 C CNN
+F 2 "Package_SO:SOP-8_3.9x4.9mm_P1.27mm" H 3800 4850 50  0001 C CNN
+F 3 "http://www.ti.com/lit/ds/symlink/lm393.pdf" H 3800 4850 50  0001 C CNN
+	3    3800 4850
 	1    0    0    -1
 $EndComp
@@
 P 5100 3100
 F 0 "R5" V 5180 3100 50  0000 C CNN
-F 1 "4.7M" V 5100 3100 50  0000 C CNN
+F 1 "102k" V 5100 3100 50  0000 C CNN
 F 2 "Resistor_SMD:R_0603_1608Metric_Pad0.98x0.95mm_HandSolder" V 5030 3100 50  0001 C CNN
 F 3 "~" H 5100 3100 50  0001 C CNN
@@
 L power:VCC #PWR0105
 U 1 1 616DD23D
-P 4350 3850
-F 0 "#PWR0105" H 4350 3700 50  0001 C CNN
-F 1 "VCC" H 4350 4000 50  0000 C CNN
-F 2 "" H 4350 3850 50  0001 C CNN
-F 3 "" H 4350 3850 50  0001 C CNN
-	1    4350 3850
+P 4350 4050
+F 0 "#PWR0105" H 4350 3900 50  0001 C CNN
+F 1 "VCC" H 4350 4200 50  0000 C CNN
+F 2 "" H 4350 4050 50  0001 C CNN
+F 3 "" H 4350 4050 50  0001 C CNN
+	1    4350 4050
 	-1   0    0    1
 $EndComp
 Wire Wire Line
-	4350 3850 4350 3800
+	4350 4050 4350 3800
 Wire Wire Line
 	4350 3800 4400 3800
@@
 L power:VCC #PWR0106
 U 1 1 616E7989
-P 3700 4300
-F 0 "#PWR0106" H 3700 4150 50  0001 C CNN
-F 1 "VCC" H 3700 4450 50  0000 C CNN
-F 2 "" H 3700 4300 50  0001 C CNN
-F 3 "" H 3700 4300 50  0001 C CNN
-	1    3700 4300
+P 3700 4500
+F 0 "#PWR0106" H 3700 4350 50  0001 C CNN
+F 1 "VCC" H 3700 4650 50  0000 C CNN
+F 2 "" H 3700 4500 50  0001 C CNN
+F 3 "" H 3700 4500 50  0001 C CNN
+	1    3700 4500
 	1    0    0    -1
 $EndComp
@@
 L power:GND #PWR0107
 U 1 1 616E80C0
-P 3700 5000
-F 0 "#PWR0107" H 3700 4750 50  0001 C CNN
-F 1 "GND" H 3700 4850 50  0000 C CNN
-F 2 "" H 3700 5000 50  0001 C CNN
-F 3 "" H 3700 5000 50  0001 C CNN
-	1    3700 5000
-	1    0    0    -1
-$EndComp
-Wire Wire Line
-	3700 5000 3700 4950
-Wire Wire Line
-	3700 4300 3700 4350
+P 3700 5200
+F 0 "#PWR0107" H 3700 4950 50  0001 C CNN
+F 1 "GND" H 3700 5050 50  0000 C CNN
+F 2 "" H 3700 5200 50  0001 C CNN
+F 3 "" H 3700 5200 50  0001 C CNN
+	1    3700 5200
+	1    0    0    -1
+$EndComp
+Wire Wire Line
+	3700 5200 3700 5150
+Wire Wire Line
+	3700 4500 3700 4550
 $Comp
 L Device:C C1
 U 1 1 616E9949
-P 3400 4650
-F 0 "C1" H 3425 4750 50  0000 L CNN
-F 1 "100n" H 3425 4550 50  0000 L CNN
-F 2 "Capacitor_SMD:C_0805_2012Metric_Pad1.18x1.45mm_HandSolder" H 3438 4500 50  0001 C CNN
-F 3 "~" H 3400 4650 50  0001 C CNN
-	1    3400 4650
-	1    0    0    -1
-$EndComp
-Wire Wire Line
-	3400 4500 3400 4350
-Wire Wire Line
-	3400 4350 3700 4350
-Connection ~ 3700 4350
-Wire Wire Line
-	3400 4800 3400 4950
-Wire Wire Line
-	3400 4950 3700 4950
-Connection ~ 3700 4950
+P 3400 4850
+F 0 "C1" H 3425 4950 50  0000 L CNN
+F 1 "100n" H 3425 4750 50  0000 L CNN
+F 2 "Capacitor_SMD:C_0805_2012Metric_Pad1.18x1.45mm_HandSolder" H 3438 4700 50  0001 C CNN
+F 3 "~" H 3400 4850 50  0001 C CNN
+	1    3400 4850
+	1    0    0    -1
+$EndComp
+Wire Wire Line
+	3400 4700 3400 4550
+Wire Wire Line
+	3400 4550 3700 4550
+Connection ~ 3700 4550
+Wire Wire Line
+	3400 5000 3400 5150
+Wire Wire Line
+	3400 5150 3700 5150
+Connection ~ 3700 5150
 $Comp
 L power:GND #PWR0108
 U 1 1 6170117A
-P 4300 5000
-F 0 "#PWR0108" H 4300 4750 50  0001 C CNN
-F 1 "GND" H 4300 4850 50  0000 C CNN
-F 2 "" H 4300 5000 50  0001 C CNN
-F 3 "" H 4300 5000 50  0001 C CNN
-	1    4300 5000
-	1    0    0    -1
-$EndComp
-Wire Wire Line
-	4300 5000 4300 4900
+P 4300 5200
+F 0 "#PWR0108" H 4300 4950 50  0001 C CNN
+F 1 "GND" H 4300 5050 50  0000 C CNN
+F 2 "" H 4300 5200 50  0001 C CNN
+F 3 "" H 4300 5200 50  0001 C CNN
+	1    4300 5200
+	1    0    0    -1
+$EndComp
+Wire Wire Line
+	4300 5200 4300 5100
+Wire Wire Line
+	4300 5100 4350 5100
+Wire Wire Line
+	4300 5100 4300 4900
 Wire Wire Line
 	4300 4900 4350 4900
-Wire Wire Line
-	4300 4900 4300 4700
-Wire Wire Line
-	4300 4700 4350 4700
-Connection ~ 4300 4900
+Connection ~ 4300 5100
 $Comp
 L power:GND #PWR0109
 U 1 1 61702A75
-P 5100 5000
-F 0 "#PWR0109" H 5100 4750 50  0001 C CNN
-F 1 "GND" H 5100 4850 50  0000 C CNN
-F 2 "" H 5100 5000 50  0001 C CNN
-F 3 "" H 5100 5000 50  0001 C CNN
-	1    5100 5000
-	1    0    0    -1
-$EndComp
-Wire Wire Line
-	4950 4800 5100 4800
-Wire Wire Line
-	5100 4800 5100 5000
+P 5100 5200
+F 0 "#PWR0109" H 5100 4950 50  0001 C CNN
+F 1 "GND" H 5100 5050 50  0000 C CNN
+F 2 "" H 5100 5200 50  0001 C CNN
+F 3 "" H 5100 5200 50  0001 C CNN
+	1    5100 5200
+	1    0    0    -1
+$EndComp
+Wire Wire Line
+	4950 5000 5100 5000
+Wire Wire Line
+	5100 5000 5100 5200
 $Comp
 L Connector_Generic:Conn_01x04 J1
@@
 	3700 3350 4100 3350
 $Comp
-L Device:Jumper JP?
+L Device:Jumper JP1
 U 1 1 616C83B1
 P 4900 2250
-F 0 "JP?" H 4900 2400 50  0000 C CNN
+F 0 "JP1" H 4900 2400 50  0000 C CNN
 F 1 "Comparitor Bypass" H 4900 2170 50  0000 C CNN
 F 2 "Resistor_SMD:R_1206_3216Metric_Pad1.30x1.75mm_HandSolder" H 4900 2250 50  0001 C CNN
@@
 Wire Wire Line
 	5700 3450 6200 3450
+$Comp
+L Device:R R7
+U 1 1 616D737B
+P 3300 3850
+F 0 "R7" V 3380 3850 50  0000 C CNN
+F 1 "4.7M" V 3300 3850 50  0000 C CNN
+F 2 "Resistor_SMD:R_0603_1608Metric_Pad0.98x0.95mm_HandSolder" V 3230 3850 50  0001 C CNN
+F 3 "~" H 3300 3850 50  0001 C CNN
+	1    3300 3850
+	1    0    0    -1
+$EndComp
+$Comp
+L power:GND #PWR0103
+U 1 1 616E36ED
+P 3300 4050
+F 0 "#PWR0103" H 3300 3800 50  0001 C CNN
+F 1 "GND" H 3300 3900 50  0000 C CNN
+F 2 "" H 3300 4050 50  0001 C CNN
+F 3 "" H 3300 4050 50  0001 C CNN
+	1    3300 4050
+	1    0    0    -1
+$EndComp
+Wire Wire Line
+	3300 4050 3300 4000
+Wire Wire Line
+	3300 3600 3300 3700
+Connection ~ 3300 3600
 $EndSCHEMATC

Commit message: add notes to circuit
Parts:
- R7: value 4.7M -> 10M
Other:
- note added: "Bridge to bypass comparator"
- note added: "D1 is used as a light sensor.\nUse red or green with clear lense"
- note added: "R5 sets hysteresis\n"
- note added: "Sets comparitor voltage"
- note added: "Spare comparator is grounded"
- note added: "Without R7 sometimes circuit LED would \nnot react to light. Acts like a sensitivity adjustment,\ndecrease R7 to decrease sensitivity"
- moved on the sheet: C1, D1, J1, JP1, Q1, R1, R2, R3, R4, R5, R6, R7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
