File: pcb/shutter_tester.kicad_sch (KiCad schematic)
At the start: 17 parts, among them J1 Conn_01x04, Q1 MMBTA13LT3G, U1 LM393

Commit message: getting to rev b layout
Parts:
- removed JP1: Comparitor Bypass, Resistor_SMD:R_1206_3216Metric_Pad1.30x1.75mm_HandSolder, symbol Device:Jumper
- added C2: 1u, Capacitor_SMD:C_0805_2012Metric_Pad1.18x1.45mm_HandSolder, symbol Device:C
- added D2: LED, LED_SMD:LED_0805_2012Metric_Pad1.15x1.40mm_HandSolder, symbol Device:LED
- added Q2: MMBTA13LT3G, Package_TO_SOT_SMD:SOT-23, symbol Device:Q_NPN_Darlington_BEC
- added R10, R11, R12, R8, R9: 4.7M, Resistor_SMD:R_0603_1608Metric_Pad0.98x0.95mm_HandSolder, symbol Device:R
- added R13: 2k, Resistor_SMD:R_0805_2012Metric_Pad1.20x1.40mm_HandSolder, symbol Device:R
- added R14: 10k, Resistor_SMD:R_0603_1608Metric_Pad0.98x0.95mm_HandSolder, symbol Device:R
- added R17: 102k, Resistor_SMD:R_0603_1608Metric_Pad0.98x0.95mm_HandSolder, symbol Device:R
- added R18: 3k, Resistor_SMD:R_0805_2012Metric_Pad1.20x1.40mm_HandSolder, symbol Device:R
- J1: footprint Connector_PinHeader_2.54mm:PinHeader_1x04_P2.54mm_Horizontal -> Connector_PinHeader_2.54mm:PinHeader_1x04_P2.54mm_Vertical
- R2, R3, R4: footprint Resistor_SMD:R_1206_3216Metric_Pad1.30x1.75mm_HandSolder -> Resistor_SMD:R_0603_1608Metric_Pad0.98x0.95mm_HandSolder
- R7: value 10M -> 4.7M
Connections:
- net GND: now also J1.1 (Pin_1), R4.2, C2.2, Q2.2 (E), R12.2, R9.2; no longer J1.2 (Pin_2), J1.4 (Pin_4), R4.1, R7.2, U1.5 (+), U1.6 (_), U1.7
- net VCC: now also J1.4 (Pin_4), R3.1, C2.1, D2.1 (K), R13.1, R18.2; no longer J1.1 (Pin_1), R3.2
- net OUTPUT renamed OUTPUT_1
- net OUTPUT_1: now also J1.2 (Pin_2); no longer J1.3 (Pin_3)
- new net: R14.1, R17.2, U1.5 (+)
- new net: R7.2, R8.1
- new net: R8.2, R9.1
- new net: R11.2, R12.1
- new net: D2.2 (A), Q2.1 (B), R10.1
- new net: R10.2, R11.1
- new net: Q2.3 (C), R13.2, R14.2
- new net OUTPUT_2: J1.3 (Pin_3), R17.1, R18.1, U1.7
- new net Vtrig: R3.2, R4.1, U1.2 (-), U1.6 (_)
Other:
- note added: "Arduino Interface"
- note added: "Comparitor Bypass Capacitors"
- note added: "Comparitor Trigger Set"
- note added: "ERC Happy Area"
- note added: "Light Sensor 1"
- note added: "Light Sensor 2"
- note added: "Mechanical Mounting"
- note added: "R17 sets hysteresis"
- note added: "R4 and R3 sets trigger voltage Vtrig = Vcc * (R4 / (R3 + R4))"
- note added: "Without R7, R8, and R9 sometimes circuit LED would not react to light. Acts like a sensitivity adjustment, decrease R7 to decrease sensitivity. I did not have a single equivalent resistor so use three in series to get high reistance if needed or replace the remaining resistors with jumpers."
- note removed: "Bridge to bypass comparator"
- note removed: "Sets comparitor voltage"
- note removed: "Spare comparator is grounded"
- note removed: "Without R7 sometimes circuit LED would not react to light. Acts like a sensitivity adjustment, decrease R7 to decrease sensitivity"
- moved on the sheet: C1, D1, H1, H2, H3, H4, J1, Q1, R1, R2, R3, R4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

Commit message: rev a layout
Connections:
- net GND: now also J1.4 (Pin_4); no longer J1.1 (Pin_1)
- net OUTPUT_1: now also J1.3 (Pin_3); no longer J1.2 (Pin_2)
- net OUTPUT_2: now also J1.2 (Pin_2); no longer J1.3 (Pin_3)
- net VCC: now also J1.1 (Pin_1); no longer J1.4 (Pin_4)
Other:
- title: Shutter Sensor -> Shutter Timming Sensor
Changed lines of the file:
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@@
   (paper "A")
   (title_block
-    (title "Shutter Sensor")
+    (title "Shutter Timming Sensor")
     (date "2022-02-28")
     (rev "A")
@@
     (pin "2")
   )
-  (symbol (lib_id "Connector_Generic:Conn_01x04") (at 215.9 85.09 0) (mirror x) (unit 1)
-    (in_bom yes) (on_board yes)
-    (property "Reference" "J1" (id 0) (at 215.9 90.17 0))
-    (property "Value" "Conn_01x04" (id 1) (at 215.9 77.47 0))
-    (property "Footprint" "Connector_PinHeader_2.54mm:PinHeader_1x04_P2.54mm_Vertical" (id 2) (at 215.9 85.09 0)
-      (effects (font (size 1.27 1.27)) hide)
-    )
-    (property "Datasheet" "~" (id 3) (at 215.9 85.09 0)
-      (effects (font (size 1.27 1.27)) hide)
-    )
+  (symbol (lib_id "Connector_Generic:Conn_01x04") (at 215.9 82.55 0) (unit 1)
+    (in_bom yes) (on_board yes)
+    (property "Reference" "J1" (id 0) (at 215.9 77.47 0))
+    (property "Value" "Conn_01x04" (id 1) (at 215.9 90.17 0))
+    (property "Footprint" "Connector_PinHeader_2.54mm:PinHeader_1x04_P2.54mm_Vertical" (id 2) (at 215.9 82.55 0)
+      (effects (font (size 1.27 1.27)) hide)
+    )
+    (property "Datasheet" "~" (id 3) (at 215.9 82.55 0)
+      (effects (font (size 1.27 1.27)) hide)
+    )
