File: pcb/sensor/shutter_tester.kicad_pcb (KiCad board)
At the start: 2 copper layers, 53 x 42 mm, 30 parts, among them J1 Conn_01x04, Q1 MMBTA13LT3G, Q2 MMBTA13LT3G, U1 LM393

Commit message: add github link
Other:
- board text added: "github.com/sdp8483/shutter_tester"
Changed lines of the file:
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@@
     (effects (font (size 1.5 1.5) (thickness 0.214286)) (justify right))
+  )
+  (gr_text "github.com/sdp8483/shutter_tester" (at 121.7 114 -90) (layer "F.SilkS")
+    (effects (font (size 1 1) (thickness 0.15)))
   )
   (gr_text "B" (at 145.25 97.35 90) (layer "F.SilkS")
